File: Hardware/Dart Board/Dart Board.kicad_sch (KiCad schematic)
At the start: 0 parts

Commit message: yay
Other:
- added sheet ADC (adc.kicad_sch)
- added sheet Battery (battery.kicad_sch)
- added sheet Connectors (conn.kicad_sch)
- title: (none) -> Dart Board
Changed lines of the file:
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@@
 	(generator_version "9.0")
 	(paper "A4")
+	(title_block
+		(title "Dart Board")
+		(date "2026-03-04")
+		(rev "01")
+	)
+	(sheet
+		(at 53.975 75.565)
+		(size 38.1 26.67)
+		(exclude_from_sim no)
+		(in_bom yes)
+		(on_board yes)
+		(dnp no)
+		(fields_autoplaced yes)
+		(stroke
+			(width 0.1524)
+			(type solid)
+		)
+		(fill
+			(color 0 0 0 0.0000)
+		)
+		(property "Sheetname" "Battery"
+			(at 53.975 74.8534 0)
+			(effects
+				(font
+					(size 1.27 1.27)
+				)
+				(justify left bottom)
+			)
+		)
+		(property "Sheetfile" "battery.kicad_sch"
+			(at 53.975 102.8196 0)
+			(effects
+				(font
+					(size 1.27 1.27)
+				)
+				(justify left top)
+			)
+		)
+		(instances
+			(project "Dart Board"
+				(path "/1d6d0dd6-dd3e-4fbe-b34b-7dc303157c7e"
+					(page "3")
+				)
+			)
+		)
+	)
+	(sheet
+		(at 97.155 26.035)
+		(size 62.23 35.56)
+		(exclude_from_sim no)
+		(in_bom yes)
+		(on_board yes)
+		(dnp no)
+		(fields_autoplaced yes)
+		(stroke
+			(width 0.1524)
+			(type solid)
+		)
+		(fill
+			(color 0 0 0 0.0000)
+		)
+		(property "Sheetname" "ADC"
+			(at 97.155 25.3234 0)
+			(effects
+				(font
+					(size 1.27 1.27)
+				)
+				(justify left bottom)
+			)
+		)
+		(property "Sheetfile" "adc.kicad_sch"
+			(at 97.155 62.1796 0)
+			(effects
+				(font
+					(size 1.27 1.27)
+				)
+				(justify left top)
+			)
+		)
+		(instances
+			(project "Dart Board"
+				(path "/1d6d0dd6-dd3e-4fbe-b34b-7dc303157c7e"
+					(page "4")
+				)
+			)
+		)
+	)
+	(sheet
+		(at 33.655 23.495)
+		(size 38.735 26.67)
+		(exclude_from_sim no)
+		(in_bom yes)
+		(on_board yes)
+		(dnp no)
+		(fields_autoplaced yes)
+		(stroke
+			(width 0.1524)
+			(type solid)
+		)
+		(fill
+			(color 0 0 0 0.0000)
+		)
+		(property "Sheetname" "Connectors"
+			(at 33.655 22.7834 0)
+			(effects
+				(font
+					(size 1.27 1.27)
+				)
+				(justify left bottom)
+			)
+		)
+		(property "Sheetfile" "conn.kicad_sch"
+			(at 33.655 50.7496 0)
+			(effects
+				(font
+					(size 1.27 1.27)
+				)
+				(justify left top)
+			)
+		)
+		(instances
+			(project "Dart Board"
+				(path "/1d6d0dd6-dd3e-4fbe-b34b-7dc303157c7e"
+					(page "2")
+				)
+			)
+		)
+	)
 	(sheet_instances
 		(path "/"

Commit message: Piezo circuit
Other:
- added sheet Piezo sensors (piezo.kicad_sch)
Changed lines of the file:
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@@
+	)
+	(sheet
+		(at 152.654 90.17)
+		(size 21.336 17.018)
+		(exclude_from_sim no)
+		(in_bom yes)
+		(on_board yes)
+		(dnp no)
+		(fields_autoplaced yes)
+		(stroke
+			(width 0.1524)
+			(type solid)
+		)
+		(fill
+			(color 0 0 0 0.0000)
+		)
+		(property "Sheetname" "Piezo sensors"
+			(at 152.654 89.4584 0)
+			(effects
+				(font
+					(size 1.27 1.27)
+				)
+				(justify left bottom)
+			)
+		)
+		(property "Sheetfile" "piezo.kicad_sch"
+			(at 152.654 107.7726 0)
+			(effects
+				(font
+					(size 1.27 1.27)
+				)
+				(justify left top)
+			)
+		)
+		(instances
+			(project "Dart Board"
+				(path "/1d6d0dd6-dd3e-4fbe-b34b-7dc303157c7e"
+					(page "5")
+				)
+			)
+		)
 	)
 	(sheet
