File: Hardware/Dart Board/Dart Board.kicad_pcb (KiCad board)
At the start: 2 copper layers, 124 parts, among them J1 Screw_Terminal_01x02, J10 Screw_Terminal_01x02, J11 Screw_Terminal_01x02, J12 Screw_Terminal_01x02, J13 Screw_Terminal_01x02, J14 Screw_Terminal_01x02, J15 Screw_Terminal_01x02, J16 Screw_Terminal_01x02, J17 Screw_Terminal_01x02, J18 Screw_Terminal_01x02, J19 Screw_Terminal_01x02, J20 Screw_Terminal_01x02, J21 Screw_Terminal_01x02, J22 Screw_Terminal_01x02, J23 Screw_Terminal_01x02, J4 Screw_Terminal_01x02, J5 Screw_Terminal_01x02, J6 Screw_Terminal_01x02, J7 Screw_Terminal_01x02, J8 Screw_Terminal_01x02, J9 Screw_Terminal_01x02, U1 ADS1115IDGS

Commit message: Finished PCB Layout
Parts:
- removed C19, C20: 4.7nF, Capacitor_SMD:C_0805_2012Metric_Pad1.18x1.45mm_HandSolder
- removed D56, D57, D58: D_Schottky, Diode_THT:D_DO-41_SOD81_P10.16mm_Horizontal
- removed D60, D61, D62: 3.3V, Diode_SMD:D_SOD-123
- removed J20, J21, J22, J23: Screw_Terminal_01x02, TerminalBlock:TerminalBlock_MaiXu_MX126-5.0-02P_1x02_P5.00mm
- removed R1: 10k, Resistor_SMD:R_0603_1608Metric_Pad0.98x0.95mm_HandSolder
- removed R20, R21: 1M, Resistor_SMD:R_0603_1608Metric_Pad0.98x0.95mm_HandSolder
- removed U1: ADS1115IDGS, Package_SO:TSSOP-10_3x3mm_P0.5mm
- added J2: Screw_Terminal_01x02, TerminalBlock:TerminalBlock_MaiXu_MX126-5.0-02P_1x02_P5.00mm, F.Cu at (199.5, 179.5)
- added J3: Screw_Terminal_01x02, TerminalBlock:TerminalBlock_MaiXu_MX126-5.0-02P_1x02_P5.00mm, F.Cu at (214.9, 179.5)
- added REF**: MountingHole_3.2mm_M3, MountingHole:MountingHole_3.2mm_M3, F.Cu at (348.5, 183.5)
- added REF**: MountingHole_3.2mm_M3, MountingHole:MountingHole_3.2mm_M3, F.Cu at (142.0, 183.5)
- added REF**: MountingHole_3.2mm_M3, MountingHole:MountingHole_3.2mm_M3, F.Cu at (348.5, 68.5)
- added REF**: MountingHole_3.2mm_M3, MountingHole:MountingHole_3.2mm_M3, F.Cu at (142.0, 68.5)
- D36, D42, D45, D54: value D_Schottky -> 3.3V; footprint Diode_THT:D_DO-41_SOD81_P10.16mm_Horizontal -> Diode_SMD:D_SOD-123
- D38, D49, D50: value 3.3V -> D_Schottky; footprint Diode_SMD:D_SOD-123 -> Diode_THT:D_DO-41_SOD81_P10.16mm_Horizontal
- moved J4 262.3 mm to (264.5, 183.2)
- moved D1 178.2 mm to (209.5, 166.9), turned to -90 degrees
- moved J8 162.3 mm to (347.5, 150.3), turned to 90 degrees
- moved J5 154.5 mm to (303.0, 176.2), turned to 90 degrees
- moved J1 135.4 mm to (229.5, 68.0), turned to 180 degrees
- moved D21 135.0 mm to (338.5, 148.8), turned to -90 degrees
- moved J7 130.2 mm to (312.5, 157.8), turned to 90 degrees
- moved J11 127.5 mm to (347.5, 121.3), turned to 90 degrees
- moved J6 122.6 mm to (276.5, 164.8), turned to 90 degrees
- moved D30 118.7 mm to (338.5, 119.8), turned to -90 degrees
- moved D12 118.6 mm to (294.0, 174.8), turned to -90 degrees
- moved J17 117.5 mm to (152.0, 97.6), turned to -90 degrees
- moved D18 114.7 mm to (303.5, 156.3), turned to -90 degrees
- moved D54 113.8 mm to (160.5, 68.0), turned to 90 degrees
- moved J18 109.0 mm to (151.7, 82.0), turned to -90 degrees
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Connections:
- A1 pad 13: PIEZO_11 -> unconnected-(A1-P16-Pad13)
- A1 pad 14: PIEZO_12 -> PIEZO_11
- A1 pad 15: PIEZO_13 -> PIEZO_12
- A1 pad 16: unconnected-(A1-P19-Pad16) -> PIEZO_13
- A1 pad 33: unconnected-(A1-P31-Pad33) -> GPIO_43
- A1 pad 34: unconnected-(A1-P32-Pad34) -> GPIO_44
- A1 pad 38: GPIO_43 -> unconnected-(A1-RXD0/P36-Pad38)
- A1 pad 39: GPIO_44 -> unconnected-(A1-TXD0/P37-Pad39)
- C10 pad 1: PIEZO_09 -> PIEZO_10
- C11 pad 1: PIEZO_10 -> PIEZO_11
- C12 pad 1: PIEZO_11 -> PIEZO_12
- C13 pad 1: PIEZO_12 -> PIEZO_13
- C14 pad 1: PIEZO_13 -> PIEZO_14
- C15 pad 1: PIEZO_14 -> PIEZO_15
- C16 pad 1: PIEZO_15 -> PIEZO_16
- C17 pad 1: PIEZO_16 -> PIEZO_17
- C18 pad 1: PIEZO_17 -> PIEZO_18
- C4 pad 1: PIEZO_03 -> PIEZO_04
- C5 pad 1: PIEZO_04 -> PIEZO_05
- C6 pad 1: PIEZO_05 -> PIEZO_06
- C7 pad 1: PIEZO_06 -> PIEZO_07
- C8 pad 1: PIEZO_07 -> PIEZO_08
- C9 pad 1: PIEZO_08 -> PIEZO_09
- D10 pad 1: PIEZO_03 -> PIEZO_04
- D11 pad 1: PIEZO_03 -> PIEZO_04
- D12 pad 1: PIEZO_03 -> PIEZO_04
- D13 pad 1: PIEZO_04 -> PIEZO_05
- D14 pad 1: PIEZO_04 -> PIEZO_05
- D15 pad 1: PIEZO_04 -> PIEZO_05
- D16 pad 1: PIEZO_05 -> PIEZO_06
- D17 pad 1: PIEZO_05 -> PIEZO_06
- D18 pad 1: PIEZO_05 -> PIEZO_06
- D19 pad 1: PIEZO_06 -> PIEZO_07
- D20 pad 1: PIEZO_06 -> PIEZO_07
- D21 pad 1: PIEZO_06 -> PIEZO_07
- D22 pad 1: PIEZO_07 -> PIEZO_08
- D23 pad 1: PIEZO_07 -> PIEZO_08
- D24 pad 1: PIEZO_07 -> PIEZO_08
- D25 pad 1: PIEZO_08 -> PIEZO_09
- D26 pad 1: PIEZO_08 -> PIEZO_09
- D27 pad 1: PIEZO_08 -> PIEZO_09
- D28 pad 1: PIEZO_09 -> PIEZO_10
- D29 pad 1: PIEZO_09 -> PIEZO_10
- D30 pad 1: PIEZO_09 -> PIEZO_10
- D31 pad 1: PIEZO_10 -> PIEZO_11
- D32 pad 1: PIEZO_10 -> PIEZO_11
- D33 pad 1: PIEZO_10 -> PIEZO_11
- D34 pad 1: PIEZO_11 -> PIEZO_12
- D35 pad 2: Net-(D35-A) -> GND
- D36 pad 1: PIEZO_11 -> PIEZO_12
- D37 pad 1: PIEZO_12 -> PIEZO_13
- D37 pad 2: GND -> Net-(D37-A)
- D38 pad 1: PIEZO_11 -> PIEZO_13
- D39 pad 1: PIEZO_12 -> PIEZO_13
- D40 pad 1: PIEZO_13 -> PIEZO_14
- D41 pad 2: Net-(D41-A) -> GND
- D42 pad 1: PIEZO_15 -> PIEZO_14
- D42 pad 2: Net-(D42-A) -> GND
- D43 pad 1: PIEZO_16 -> PIEZO_15
- D44 pad 1: PIEZO_13 -> PIEZO_15
- D45 pad 1: PIEZO_14 -> PIEZO_15
- D46 pad 1: PIEZO_15 -> PIEZO_16
- D46 pad 2: GND -> Net-(D46-A)
- D48 pad 1: PIEZO_13 -> PIEZO_16
- D49 pad 1: PIEZO_14 -> PIEZO_17
- D49 pad 2: GND -> Net-(D49-A)
- D50 pad 1: PIEZO_15 -> PIEZO_17
- D51 pad 1: PIEZO_16 -> PIEZO_17
- D52 pad 1: PIEZO_17 -> PIEZO_18
- D53 pad 2: Net-(D53-A) -> GND
- D54 pad 1: PIEZO_19 -> PIEZO_18
- D54 pad 2: Net-(D54-A) -> GND
- J10 pad 2: Net-(D19-A) -> Net-(D25-A)
- J11 pad 2: Net-(D22-A) -> Net-(D28-A)
- J12 pad 2: Net-(D25-A) -> Net-(D31-A)
- J13 pad 2: Net-(D28-A) -> Net-(D34-A)
- J14 pad 2: Net-(D31-A) -> Net-(D37-A)
- J15 pad 2: Net-(D34-A) -> Net-(D40-A)
- J16 pad 2: Net-(D35-A) -> Net-(D43-A)
- J17 pad 2: Net-(D40-A) -> Net-(D46-A)
- J18 pad 2: Net-(D41-A) -> Net-(D49-A)
- J19 pad 2: Net-(D42-A) -> Net-(D52-A)
- J4 pad 2: Net-(D1-A) -> Net-(D7-A)
- J5 pad 2: Net-(D4-A) -> Net-(D10-A)
- J6 pad 2: Net-(D7-A) -> Net-(D13-A)
- J7 pad 2: Net-(D10-A) -> Net-(D16-A)
- J8 pad 2: Net-(D13-A) -> Net-(D19-A)
- J9 pad 2: Net-(D16-A) -> Net-(D22-A)
- R10 pad 1: PIEZO_08 -> PIEZO_09
- R11 pad 1: PIEZO_09 -> PIEZO_10
- R12 pad 1: PIEZO_10 -> PIEZO_11
- R13 pad 1: PIEZO_11 -> PIEZO_12
- R14 pad 1: PIEZO_12 -> PIEZO_13
- R15 pad 1: PIEZO_13 -> PIEZO_14
- R16 pad 1: PIEZO_14 -> PIEZO_15
- R17 pad 1: PIEZO_15 -> PIEZO_16
- R18 pad 1: PIEZO_16 -> PIEZO_17
- R19 pad 1: PIEZO_17 -> PIEZO_18
- R5 pad 1: PIEZO_03 -> PIEZO_04
- R6 pad 1: PIEZO_04 -> PIEZO_05
- R7 pad 1: PIEZO_05 -> PIEZO_06
- R8 pad 1: PIEZO_06 -> PIEZO_07
- R9 pad 1: PIEZO_07 -> PIEZO_08
Routing:
- net GND: track 0.00 -> 347.9 mm
- net PIEZO_07: track 0.00 -> 166.2 mm
- net PIEZO_10: track 0.00 -> 142.0 mm
- net PIEZO_04: track 0.00 -> 139.5 mm
- net PIEZO_06: track 0.00 -> 134.1 mm
- net PIEZO_13: track 0.00 -> 132.9 mm
- net PIEZO_09: track 0.00 -> 112.0 mm
- net PIEZO_03: track 0.00 -> 106.6 mm
- net PIEZO_05: track 0.00 -> 100.4 mm
- net PIEZO_12: track 0.00 -> 96.9 mm
- net PIEZO_15: track 0.00 -> 94.2 mm
- net PIEZO_01: track 0.00 -> 87.4 mm
- net PIEZO_08: track 0.00 -> 81.7 mm
- net PIEZO_02: track 0.00 -> 79.9 mm
- net PIEZO_11: track 0.00 -> 63.3 mm
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- added copper zone on B.Cu, net GND
Other:
- board outline added: 218.5 x 127 mm
